File: kicad/ckt-katoswitch/ckt-katoswitch.kicad_sch (KiCad schematic)
At the start: 39 parts, among them J1 Screw_Terminal_01x02, J2 Screw_Terminal_01x02, J3 Conn_AVR_TagConnect_TC2030, J4 Screw_Terminal_01x02, J5 Screw_Terminal_01x02, J6 Screw_Terminal_01x02, K1 AGQ200A4H, Q1 DRDC3105-7, U1 AP7381-50Y, U2 DRV8231A, U3 ATtiny414-SS, U4 LTV-357T

Commit message: Add touch-toggle header since that's apparently common on T-Trak
Parts:
- added J7: Conn_01x03, symbol Connector_Generic:Conn_01x03
Connections:
- net +5V: now also J7.2 (Pin_2)
- net GND: now also J7.3 (Pin_3)
- net at C6.1, J6.1 (Pin_1), R3.2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: now also J7.1 (Pin_1)
Other:
- note added: "Touch Toggle Interface Level-triggered option must be soldered"
- moved on the sheet: C1, C2, C3, C4, C5, C6, C7, D1, D2, D3, D4, D5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

Commit message: Initial cut at PCB
Parts:
- removed C5: 1uF, Capacitor_SMD:C_0805_2012Metric, symbol Device:C
- J7: footprint (none) -> Connector_PinHeader_2.54mm:PinHeader_1x03_P2.54mm_Vertical
- renumbered D2 to D1, D1 to D2, D4 to D3, D3 to D4
Connections:
- net at J6.1 (Pin_1), J7.1 (Pin_1), R3.2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: no longer C6.1
- net at R5.1, U3.12 (PA2): now also C7.1
- net at D8.2 (A), J6.3 (Pin_3), R5.2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: no longer C7.1
- net at JP1.2 (B): now also U3.8 (PB1); no longer U3.3 (PA5)
- net at R4.1, U3.11 (PA1), U4.4: now also C6.1
- net at JP3.2 (B): now also U3.6 (PB3); no longer U3.5 (PA7)
- net at Q1.1 (G): now also U3.4 (PA6); no longer U3.7 (PB2)
- net at JP2.2 (B): now also U3.7 (PB2); no longer U3.4 (PA6)
- net at U3.2 (PA4): now also U2.2 (IN2)
- net GATE_X1: no longer names the net of U2.3 (IN1)
- net GATE_X1: now also U3.3 (PA5); no longer U3.9 (PB0)
- removed net GATE_X2: U2.2 (IN2), U3.8 (PB1)
Other:
- moved on the sheet: C6, C7, R4, R5

Commit message: Updates to add "switch reverse" indicator
Parts:
- added D9: AMBER, LED_SMD:LED_0805_2012Metric, symbol Device:LED
- added R6: 1k, Resistor_SMD:R_0805_2012Metric, symbol Device:R_US
- R1: value 1k -> 10k
Connections:
- net GND: now also D9.1 (K)
- net at Q1.1 (G), U3.4 (PA6): now also R6.1
- new net: D9.2 (A), R6.2
Changed lines of the file:
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@@
 	)
 	(junction
+		(at 171.45 133.35)
+		(diameter 0)
+		(color 0 0 0 0)
+	)
+	(junction
 		(at 222.25 59.69)
 		(diameter 0)
@@
 	(wire
 		(pts
+			(xy 171.45 148.59) (xy 171.45 147.32)
+		)
+		(stroke
+			(width 0)
+			(type default)
+		)
+	)
+	(wire
+		(pts
 			(xy 68.58 120.65) (xy 68.58 123.19)
 		)
@@
 	(wire
 		(pts
+			(xy 171.45 157.48) (xy 171.45 156.21)
+		)
+		(stroke
+			(width 0)
+			(type default)
+		)
+	)
+	(wire
+		(pts
 			(xy 210.82 55.88) (xy 208.28 55.88)
 		)
@@
 	(wire
 		(pts
+			(xy 171.45 133.35) (xy 171.45 139.7)
+		)
+		(stroke
+			(width 0)
+			(type default)
+		)
+	)
+	(wire
+		(pts
 			(xy 96.52 130.81) (xy 101.6 130.81)
 		)
@@
 			)
 		)
-		(property "Value" "1k"
+		(property "Value" "10k"
 			(at 140.335 53.34 0)
 			(effects
@@
 	)
 	(symbol
+		(lib_id "Device:R_US")
+		(at 171.45 143.51 0)
+		(unit 1)
+		(exclude_from_sim no)
+		(in_bom yes)
+		(on_board yes)
+		(dnp no)
+		(property "Reference" "R6"
+			(at 166.878 142.494 0)
+			(effects
+				(font
+					(size 1.27 1.27)
+				)
+				(justify left)
+			)
+		)
+		(property "Value" "1k"
+			(at 167.005 144.272 0)
+			(effects
+				(font
+					(size 1.27 1.27)
+				)
+				(justify left)
+			)
+		)
+		(property "Footprint" "Resistor_SMD:R_0805_2012Metric"
+			(at 172.466 143.764 90)
+			(effects
+				(font
+					(size 1.27 1.27)
+				)
+				(hide yes)
+			)
+		)
+		(property "Datasheet" "~"
+			(at 171.45 143.51 0)
+			(effects
+				(font
+					(size 1.27 1.27)
+				)
+				(hide yes)
+			)
+		)
+		(property "Description" ""
+			(at 171.45 143.51 0)
+			(effects
+				(font
+					(size 1.27 1.27)
+				)
+			)
+		)
+		(pin "1"
+		)
+		(pin "2"
+		)
+		(instances
+			(project "ckt-katoswitch"
+				(path "/ee2a1513-8489-42c3-8daf-9d032b383b2d"
+					(reference "R6")
+					(unit 1)
+				)
+			)
+		)
+	)
+	(symbol
+		(lib_id "power:GND")
+		(at 171.45 157.48 0)
+		(mirror y)
+		(unit 1)
+		(exclude_from_sim no)
+		(in_bom yes)
+		(on_board yes)
+		(dnp no)
+		(property "Reference" "#PWR012"
+			(at 171.45 163.83 0)
+			(effects
+				(font
+					(size 1.27 1.27)
+				)
+				(hide yes)
+			)
+		)
+		(property "Value" "GND"
+			(at 171.45 161.29 0)
+			(effects
+				(font
+					(size 1.27 1.27)
+				)
+				(hide yes)
+			)
+		)
+		(property "Footprint" ""
+			(at 171.45 157.48 0)
+			(effects
+				(font
+					(size 1.27 1.27)
+				)
+				(hide yes)
+			)
+		)
+		(property "Datasheet" ""
+			(at 171.45 157.48 0)
+			(effects
+				(font
+					(size 1.27 1.27)
+				)
+				(hide yes)
+			)
+		)
+		(property "Description" ""
+			(at 171.45 157.48 0)
+			(effects
+				(font
+					(size 1.27 1.27)
+				)
+			)
+		)
+		(pin "1"
+		)
+		(instances
+			(project "ckt-katoswitch"
+				(path "/ee2a1513-8489-42c3-8daf-9d032b383b2d"
+					(reference "#PWR012")
+					(unit 1)
+				)
+			)
+		)
+	)
+	(symbol
 		(lib_id "Jumper:SolderJumper_2_Open")
 		(at 115.57 146.05 90)
@@
 					(unit 1)
 				)
+			)
+		)
+	)
+	(symbol
+		(lib_id "Device:LED")
+		(at 171.45 152.4 90)
+		(unit 1)
+		(exclude_from_sim no)
+		(in_bom yes)
+		(on_board yes)
+		(dnp no)
+		(property "Reference" "D9"
+			(at 172.72 149.86 90)
+			(effects
+				(font
+					(size 1.27 1.27)
+				)
+				(justify right)
+			)
+		)
+		(property "Value" "AMBER"
+			(at 176.022 151.13 0)
+			(effects
+				(font
+					(size 1.27 1.27)
+				)
+				(justify right)
+			)
+		)
+		(property "Footprint" "LED_SMD:LED_0805_2012Metric"
+			(at 171.45 152.4 0)
+			(effects
+				(font
+					(size 1.27 1.27)
+				)
+				(hide yes)
+			)
+		)
+		(property "Datasheet" "~"
+			(at 171.45 152.4 0)
+			(effects
+				(font
+					(size 1.27 1.27)
+				)
+				(hide yes)
+			)
+		)
+		(property "Description" ""
+			(at 171.45 152.4 0)
+			(effects
+				(font
+					(size 1.27 1.27)
+				)
+			)
+		)
+		(pin "1"
+		)
+		(pin "2"
+		)
+		(instances
+			(project "ckt-katoswitch"
+				(path "/ee2a1513-8489-42c3-8daf-9d032b383b2d"
+					(reference "D9")
+					(unit 1)
+				)
